File: SHMod24.kicad_pcb (KiCad board)
At the start: 2 copper layers, 49.5 x 49.5 mm, 42 parts, among them IC1 ArduinoProMini, J1 Conn_02x14_Odd_Even, J2 Conn_01x01, J3 Conn_01x01, J5 12V, Q1 FS8205A, U1 ESP-12, U2 NRF24L01, U3 AP2112K-3.3, U4 TP4056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

Commit message: add holes
Parts:
- added ?: MountingHole_3.2mm_M3, MountingHole:MountingHole_3.2mm_M3, F.Cu at (76.2, 65.4)
- added ?: MountingHole_3.2mm_M3, MountingHole:MountingHole_3.2mm_M3, F.Cu at (54.0, 108.6)
- added ?: MountingHole_3.2mm_M3, MountingHole:MountingHole_3.2mm_M3, F.Cu at (97.2, 108.6)
Changed lines of the file:
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@@
-(kicad_pcb (version 20171130) (host pcbnew "(5.0.0-rc2-18-g3893c43eb)")
+(kicad_pcb (version 20171130) (host pcbnew "(5.0.0-rc2-dev-744-gdfcdfe91f)")
   (general
     (thickness 1.6)
@@
     (tracks 813)
     (zones 0)
-    (modules 42)
+    (modules 45)
     (nets 55)
   )
@@
     (pad_to_mask_clearance 0.2)
     (aux_axis_origin 50.8 111.76)
-    (visible_elements 7FFFFF9F)
+    (visible_elements 7FFFFFBF)
     (pcbplotparams
       (layerselection 0x00030_80000001)
@@
     (uvia_drill 0.1)
     (add_net VCC)
+  )
+  (module MountingHole:MountingHole_3.2mm_M3 (layer F.Cu)
+    (at 76.2 65.405)
+    (descr "Mounting Hole 3.2mm, no annular, M3")
+    (tags "mounting hole 3.2mm no annular m3")
+    (attr virtual)
+    (fp_text reference "" (at 0 -4.2) (layer F.SilkS)
+      (effects (font (size 1 1) (thickness 0.15)))
+    )
+    (fp_text value MountingHole_3.2mm_M3 (at 0 4.2) (layer F.Fab)
+      (effects (font (size 1 1) (thickness 0.15)))
+    )
+    (fp_circle (center 0 0) (end 3.45 0) (layer F.CrtYd) (width 0.05))
+    (fp_circle (center 0 0) (end 3.2 0) (layer Cmts.User) (width 0.15))
+    (fp_text user %R (at 0.3 0) (layer F.Fab)
+      (effects (font (size 1 1) (thickness 0.15)))
+    )
+    (pad 1 np_thru_hole circle (at 0 0) (size 3.2 3.2) (drill 3.2) (layers *.Cu *.Mask))
+  )
+  (module MountingHole:MountingHole_3.2mm_M3 (layer F.Cu)
+    (at 53.975 108.585)
+    (descr "Mounting Hole 3.2mm, no annular, M3")
+    (tags "mounting hole 3.2mm no annular m3")
+    (attr virtual)
+    (fp_text reference "" (at 0 -4.2) (layer F.SilkS)
+      (effects (font (size 1 1) (thickness 0.15)))
+    )
+    (fp_text value MountingHole_3.2mm_M3 (at 0 4.2) (layer F.Fab)
+      (effects (font (size 1 1) (thickness 0.15)))
+    )
+    (fp_text user %R (at 0.3 0) (layer F.Fab)
+      (effects (font (size 1 1) (thickness 0.15)))
+    )
+    (fp_circle (center 0 0) (end 3.2 0) (layer Cmts.User) (width 0.15))
+    (fp_circle (center 0 0) (end 3.45 0) (layer F.CrtYd) (width 0.05))
+    (pad 1 np_thru_hole circle (at 0 0) (size 3.2 3.2) (drill 3.2) (layers *.Cu *.Mask))
   )
   (module Connector_PinHeader_2.54mm:PinHeader_2x14_P2.54mm_Vertical_SMD (layer F.Cu)
@@
     )
   )
+  (module MountingHole:MountingHole_3.2mm_M3 (layer F.Cu)
+    (at 97.155 108.585)
+    (descr "Mounting Hole 3.2mm, no annular, M3")
+    (tags "mounting hole 3.2mm no annular m3")
+    (attr virtual)
+    (fp_text reference "" (at 0 -4.2) (layer F.SilkS)
+      (effects (font (size 1 1) (thickness 0.15)))
+    )
+    (fp_text value MountingHole_3.2mm_M3 (at 0 4.2) (layer F.Fab)
+      (effects (font (size 1 1) (thickness 0.15)))
+    )
+    (fp_circle (center 0 0) (end 3.45 0) (layer F.CrtYd) (width 0.05))
+    (fp_circle (center 0 0) (end 3.2 0) (layer Cmts.User) (width 0.15))
+    (fp_text user %R (at 0.3 0) (layer F.Fab)
+      (effects (font (size 1 1) (thickness 0.15)))
+    )
+    (pad 1 np_thru_hole circle (at 0 0) (size 3.2 3.2) (drill 3.2) (layers *.Cu *.Mask))
+  )
   (gr_line (start 50.8 111.76) (end 50.8 62.23) (angle 90) (layer Edge.Cuts) (width 0.15))

Commit message: minor changes
Parts:
- removed ? (x3): MountingHole_3.2mm_M3, MountingHole:MountingHole_3.2mm_M3
- added J4: RESET, TestPoint:TestPoint_Pad_D1.0mm, B.Cu at (73.3, 72.9)
- added J6: GND, TestPoint:TestPoint_Pad_D1.0mm, B.Cu at (73.3, 71.8)
- added MK1: Mounting_Hole, MountingHole:MountingHole_3.2mm_M3, F.Cu at (75.6, 65.4)
- added MK2: Mounting_Hole, MountingHole:MountingHole_3.2mm_M3, F.Cu at (54.0, 108.6)
- added MK3: Mounting_Hole, MountingHole:MountingHole_3.2mm_M3, F.Cu at (97.2, 108.6)
Routing:
- net +BATT: track 51.5 -> 48.3 mm
- net Net-(J4-Pad1): track 6.22 -> 7.62 mm
- net P10: track 33.8 -> 32.5 mm
- net GND: track 80.7 -> 81.8 mm, vias 7 -> 8
- net GPIO0: track 83.3 -> 82.3 mm
- net GPIO14: track 67.7 -> 67.0 mm
