File: SHMod24.kicad_pcb (KiCad board)
At the start: 2 copper layers, 49.5 x 49.5 mm, 73 parts, among them IC1 ArduinoProMini, J1 Conn_02x14_Odd_Even, J2 Conn_01x01, J3 Conn_01x01, J4 RESET, J5 12V, J6 GND, J8 GND, J9 Screw_Terminal_01x02, Q1 FS8205A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

Commit message: final touches & gerber files
Parts:
- moved SYM1 4.21 mm to (77.0, 72.4)
Changed lines of the file:
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@@
     (thickness 1.6)
     (drawings 15)
-    (tracks 1112)
+    (tracks 1110)
     (zones 0)
     (modules 73)
@@
     (visible_elements 7FFDFFFF)
     (pcbplotparams
-      (layerselection 0x00030_80000001)
+      (layerselection 0x010f0_ffffffff)
       (usegerberextensions false)
       (usegerberattributes false)
@@
       (outputformat 1)
       (mirror false)
-      (drillshape 1)
+      (drillshape 0)
       (scaleselection 1)
-      (outputdirectory ""))
+      (outputdirectory gerber/))
   )
   (net 0 "")
@@
   )
   (module leodj-kicad:Otter_Lightbulb_smaller (layer F.Cu)
-    (at 72.771 72.009)
+    (at 76.962 72.39)
     (fp_text reference SYM1 (at 0 0) (layer F.SilkS) hide
       (effects (font (size 1.524 1.524) (thickness 0.3)))
@@
     (descr "Terminal Block Phoenix MPT-0,5-2-2.54, 2 pins, pitch 2.54mm, size 5.54x6.2mm^2, drill diamater 1.1mm, pad diameter 2.2mm, see http://www.mouser.com/ds/2/324/ItemDetail_1725656-920552.pdf, script-generated using https://github.com/pointhi/kicad-footprint-generator/scripts/TerminalBlock_Phoenix")
     (tags "THT Terminal Block Phoenix MPT-0.5-2-2.54 pitch 2.54mm size 5.54x6.2mm^2 drill 1.1mm pad 2.2mm")
-    (fp_text reference J9 (at 1.27 4.16 90) (layer B.SilkS)
+    (fp_text reference J9 (at 4.826 -2.159 180) (layer B.SilkS)
       (effects (font (size 1 1) (thickness 0.15)) (justify mirror))
     )
@@
   (segment (start 68.9915 109.347) (end 68.326 109.347) (width 0.8) (layer B.Cu) (net 16))
   (segment (start 68.326 109.347) (end 67.192 108.213) (width 0.8) (layer B.Cu) (net 16))
-  (segment (start 68.9915 109.347) (end 70.5665 109.347) (width 0.8) (layer B.Cu) (net 16))
-  (segment (start 70.5665 109.347) (end 71.0745 109.855) (width 0.8) (layer B.Cu) (net 16))
-  (segment (start 71.266501 110.047001) (end 76.881041 110.047001) (width 0.4) (layer B.Cu) (net 16))
-  (segment (start 76.881041 110.047001) (end 77.073042 109.855) (width 0.4) (layer B.Cu) (net 16))
-  (segment (start 71.0745 109.855) (end 71.266501 110.047001) (width 0.4) (layer B.Cu) (net 16))
   (segment (start 56.007 105.156) (end 55.626 104.775) (width 0.8) (layer B.Cu) (net 16))
   (segment (start 56.007 106.172) (end 56.007 105.156) (width 0.8) (layer B.Cu) (net 16))
@@
   (segment (start 76.28 88.599) (end 78.74 91.059) (width 0.4) (layer B.Cu) (net 16))
   (segment (start 76.28 88.011) (end 76.28 88.599) (width 0.4) (layer B.Cu) (net 16))
-  (segment (start 77.073042 109.855) (end 77.216 109.855) (width 0.8) (layer B.Cu) (net 16))
   (via (at 83.439 103.632) (size 0.6) (drill 0.4) (layers F.Cu B.Cu) (net 16))
   (via (at 83.439 102.997) (size 0.6) (drill 0.4) (layers F.Cu B.Cu) (net 16))
-  (segment (start 77.216 109.855) (end 83.439 103.632) (width 0.8) (layer B.Cu) (net 16))
   (segment (start 83.439 103.632) (end 83.439 102.997) (width 0.8) (layer B.Cu) (net 16))
   (segment (start 83.40999 101.18999) (end 82.976999 100.756999) (width 0.8) (layer F.Cu) (net 16))
@@
   (segment (start 82.677 100.457) (end 82.677008 100.457) (width 0.8) (layer B.Cu) (net 16))
   (segment (start 83.439 102.997) (end 83.439 103.632) (width 0.8) (layer F.Cu) (net 16))
+  (segment (start 77.216 109.855) (end 83.439 103.632) (width 0.8) (layer B.Cu) (net 16))
+  (segment (start 76.708 110.363) (end 77.216 109.855) (width 0.8) (layer B.Cu) (net 16))
+  (segment (start 71.5825 110.363) (end 76.708 110.363) (width 0.8) (layer B.Cu) (net 16))
+  (segment (start 70.5665 109.347) (end 71.5825 110.363) (width 0.8) (layer B.Cu) (net 16))
+  (segment (start 68.9915 109.347) (end 70.5665 109.347) (width 0.8) (layer B.Cu) (net 16))
   (segment (start 67.056 103.139) (end 67.056 102.064) (width 0.25) (layer F.Cu) (net 17))
   (segment (start 78.095 72.517) (end 77.978 72.4) (width 0.25) (layer B.Cu) (net 17))
