File: SHMod24.sch (KiCad schematic (older format))
At the start: 34 parts, among them IC1 ArduinoProMini, J1 Conn_01x01, J2 Conn_01x01, J3 Conn_01x01, J4 Conn_01x01, Q1 FS8205A, U1 ESP-12, U2 NRF24L01, U3 AP2112K-3.3, U4 TP4056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

Commit message: include footprints
Parts:
- added J5: 12V, symbol Screw_Terminal_01x02
Changed lines of the file:
@@
 EESchema Schematic File Version 2
-LIBS:SHMod24-rescue
 LIBS:power
 LIBS:device
@@
 LIBS:valves
 LIBS:ESP8266
-LIBS:arduino
 LIBS:mysensors_arduino
 LIBS:mysensors_connectors
@@
 LIBS:mysensors_security
 LIBS:mysensors_sensors
-LIBS:LeoDJ-lib
+LIBS:LeoDJ-kicad
 LIBS:SHMod24-cache
 EELAYER 25 0
@@
 SCK
 $Comp
-L GND #PWR01
+L GND #PWR33
 U 1 1 5ADE514E
 P 9700 2750
-F 0 "#PWR01" H 9700 2500 50  0001 C CNN
+F 0 "#PWR33" H 9700 2500 50  0001 C CNN
 F 1 "GND" H 9700 2600 50  0000 C CNN
 F 2 "" H 9700 2750 50  0001 C CNN
@@
 $EndComp
 $Comp
-L +3V3 #PWR02
+L +3V3 #PWR32
 U 1 1 5ADE517E
 P 9700 1700
-F 0 "#PWR02" H 9700 1550 50  0001 C CNN
+F 0 "#PWR32" H 9700 1550 50  0001 C CNN
 F 1 "+3V3" H 9700 1840 50  0000 C CNN
 F 2 "" H 9700 1700 50  0001 C CNN
@@
 SCL
 $Comp
-L GND #PWR03
+L GND #PWR24
 U 1 1 5ADE53C9
 P 5350 3900
-F 0 "#PWR03" H 5350 3650 50  0001 C CNN
+F 0 "#PWR24" H 5350 3650 50  0001 C CNN
 F 1 "GND" H 5350 3750 50  0000 C CNN
 F 2 "" H 5350 3900 50  0001 C CNN
@@
 $EndComp
 $Comp
-L GND #PWR04
+L GND #PWR17
 U 1 1 5ADE54F9
 P 2950 3300
-F 0 "#PWR04" H 2950 3050 50  0001 C CNN
+F 0 "#PWR17" H 2950 3050 50  0001 C CNN
 F 1 "GND" H 2950 3150 50  0000 C CNN
 F 2 "" H 2950 3300 50  0001 C CNN
@@
 $EndComp
 $Comp
-L +3V3 #PWR05
+L +3V3 #PWR1
 U 1 1 5AE0DD10
 P 650 2050
-F 0 "#PWR05" H 650 1900 50  0001 C CNN
+F 0 "#PWR1" H 650 1900 50  0001 C CNN
 F 1 "+3V3" H 650 2190 50  0000 C CNN
 F 2 "" H 650 2050 50  0001 C CNN
@@
 $EndComp
 $Comp
-L GND #PWR06
+L GND #PWR4
 U 1 1 5AE0E585
 P 1200 1850
-F 0 "#PWR06" H 1200 1600 50  0001 C CNN
+F 0 "#PWR4" H 1200 1600 50  0001 C CNN
 F 1 "GND" H 1200 1700 50  0000 C CNN
 F 2 "" H 1200 1850 50  0001 C CNN
@@
 $EndComp
 $Comp
-L +BATT #PWR07
+L +BATT #PWR8
 U 1 1 5AE60107
 P 1500 3950
-F 0 "#PWR07" H 1500 3800 50  0001 C CNN
+F 0 "#PWR8" H 1500 3800 50  0001 C CNN
 F 1 "+BATT" H 1500 4090 50  0000 C CNN
 F 2 "" H 1500 3950 50  0001 C CNN
@@
 $EndComp
 $Comp
-L +3.3V #PWR08
+L +3.3V #PWR9
 U 1 1 5AE601A7
 P 1500 4200
-F 0 "#PWR08" H 1500 4050 50  0001 C CNN
+F 0 "#PWR9" H 1500 4050 50  0001 C CNN
 F 1 "+3.3V" H 1500 4340 50  0000 C CNN
 F 2 "" H 1500 4200 50  0001 C CNN
@@
 $EndComp
 $Comp
-L GND #PWR09
+L GND #PWR10
 U 1 1 5AE601D9
 P 1500 4450
-F 0 "#PWR09" H 1500 4200 50  0001 C CNN
+F 0 "#PWR10" H 1500 4200 50  0001 C CNN
 F 1 "GND" H 1500 4300 50  0000 C CNN
 F 2 "" H 1500 4450 50  0001 C CNN
@@
 $EndComp
 $Comp
-L +3.3V #PWR010
+L +3.3V #PWR34
 U 1 1 5AE60529
 P 10500 5450
-F 0 "#PWR010" H 10500 5300 50  0001 C CNN
+F 0 "#PWR34" H 10500 5300 50  0001 C CNN
 F 1 "+3.3V" H 10500 5590 50  0000 C CNN
 F 2 "" H 10500 5450 50  0001 C CNN
@@
 $EndComp
 $Comp
-L +VDC #PWR011
+L +VDC #PWR7
 U 1 1 5AE60D76
 P 1500 3700
-F 0 "#PWR011" H 1500 3600 50  0001 C CNN
+F 0 "#PWR7" H 1500 3600 50  0001 C CNN
 F 1 "+VDC" H 1500 3950 50  0000 C CNN
 F 2 "" H 1500 3700 50  0001 C CNN
@@
 A0
 $Comp
-L +3.3V #PWR012
+L +3.3V #PWR22
 U 1 1 5AE61D43
 P 5200 1400
-F 0 "#PWR012" H 5200 1250 50  0001 C CNN
+F 0 "#PWR22" H 5200 1250 50  0001 C CNN
 F 1 "+3.3V" H 5200 1540 50  0000 C CNN
 F 2 "" H 5200 1400 50  0001 C CNN
@@
 $EndComp
 $Comp
-L +3V3 #PWR013
+L +3V3 #PWR16
 U 1 1 5AE631B5
 P 2950 1500
-F 0 "#PWR013" H 2950 1350 50  0001 C CNN
+F 0 "#PWR16" H 2950 1350 50  0001 C CNN
 F 1 "+3V3" H 2950 1640 50  0000 C CNN
 F 2 "" H 2950 1500 50  0001 C CNN
@@
 $EndComp
 $Comp
-L GND #PWR014
+L GND #PWR19
 U 1 1 5AE66520
 P 3750 7500
-F 0 "#PWR014" H 3750 7250 50  0001 C CNN
+F 0 "#PWR19" H 3750 7250 50  0001 C CNN
 F 1 "GND" H 3750 7350 50  0000 C CNN
 F 2 "" H 3750 7500 50  0001 C CNN
@@
 $EndComp
 $Comp
-L +BATT #PWR015
+L +BATT #PWR18
 U 1 1 5AE66BB8
 P 3500 5700
-F 0 "#PWR015" H 3500 5550 50  0001 C CNN
+F 0 "#PWR18" H 3500 5550 50  0001 C CNN
 F 1 "+BATT" H 3500 5840 50  0000 C CNN
 F 2 "" H 3500 5700 50  0001 C CNN
@@
 $EndComp
 $Comp
-L -BATT #PWR016
+L -BATT #PWR15
 U 1 1 5AE66C0B
 P 2500 7500
-F 0 "#PWR016" H 2500 7350 50  0001 C CNN
+F 0 "#PWR15" H 2500 7350 50  0001 C CNN
 F 1 "-BATT" H 2500 7640 50  0000 C CNN
 F 2 "" H 2500 7500 50  0001 C CNN
@@
 $EndComp
 $Comp
-L GND #PWR017
+L GND #PWR2
 U 1 1 5AE67257
 P 800 7550
-F 0 "#PWR017" H 800 7300 50  0001 C CNN
+F 0 "#PWR2" H 800 7300 50  0001 C CNN
 F 1 "GND" H 800 7400 50  0000 C CNN
 F 2 "" H 800 7550 50  0001 C CNN
@@
 $EndComp
 $Comp
-L +5V #PWR018
+L +5V #PWR3
 U 1 1 5AE67431
 P 900 7550
-F 0 "#PWR018" H 900 7400 50  0001 C CNN
+F 0 "#PWR3" H 900 7400 50  0001 C CNN
 F 1 "+5V" H 900 7690 50  0000 C CNN
 F 2 "" H 900 7550 50  0001 C CNN
@@
 $EndComp
 $Comp
-L +5V #PWR019
+L +5V #PWR11
 U 1 1 5AE67716
 P 2000 6800
-F 0 "#PWR019" H 2000 6650 50  0001 C CNN
+F 0 "#PWR11" H 2000 6650 50  0001 C CNN
 F 1 "+5V" H 2000 6940 50  0000 C CNN
 F 2 "" H 2000 6800 50  0001 C CNN
@@
 $EndComp
 $Comp
-L +BATT #PWR020
+L +BATT #PWR14
 U 1 1 5AE67751
 P 2250 7450
-F 0 "#PWR020" H 2250 7300 50  0001 C CNN
+F 0 "#PWR14" H 2250 7300 50  0001 C CNN
 F 1 "+BATT" H 2250 7590 50  0000 C CNN
 F 2 "" H 2250 7450 50  0001 C CNN
@@
 $EndComp
 $Comp
-L GND #PWR021
+L GND #PWR13
 U 1 1 5AE67CA4
 P 2250 6950
-F 0 "#PWR021" H 2250 6700 50  0001 C CNN
+F 0 "#PWR13" H 2250 6700 50  0001 C CNN
 F 1 "GND" H 2250 6800 50  0000 C CNN
 F 2 "" H 2250 6950 50  0001 C CNN
@@
 $EndComp
 $Comp
-L +BATT #PWR022
+L +BATT #PWR12
 U 1 1 5AE67DDE
 P 2250 6650
-F 0 "#PWR022" H 2250 6500 50  0001 C CNN
+F 0 "#PWR12" H 2250 6500 50  0001 C CNN
 F 1 "+BATT" H 2250 6790 50  0000 C CNN
 F 2 "" H 2250 6650 50  0001 C CNN
@@
 $EndComp
 $Comp
-L +5V #PWR023
+L +5V #PWR30
 U 1 1 5AE69210
 P 8000 5250
-F 0 "#PWR023" H 8000 5100 50  0001 C CNN
+F 0 "#PWR30" H 8000 5100 50  0001 C CNN
 F 1 "+5V" H 8000 5390 50  0000 C CNN
 F 2 "" H 8000 5250 50  0001 C CNN
@@
 $EndComp
 $Comp
-L +BATT #PWR024
+L +BATT #PWR31
 U 1 1 5AE69252
 P 8950 5250
-F 0 "#PWR024" H 8950 5100 50  0001 C CNN
+F 0 "#PWR31" H 8950 5100 50  0001 C CNN
 F 1 "+BATT" H 8950 5390 50  0000 C CNN
 F 2 "" H 8950 5250 50  0001 C CNN
@@
 	5000 6050 5000 6150
 $Comp
-L GND #PWR025
+L GND #PWR20
 U 1 1 5AEB7DAF
 P 4050 6150
-F 0 "#PWR025" H 4050 5900 50  0001 C CNN
+F 0 "#PWR20" H 4050 5900 50  0001 C CNN
 F 1 "GND" H 4050 6000 50  0000 C CNN
 F 2 "" H 4050 6150 50  0001 C CNN
@@
 $EndComp
 $Comp
-L GND #PWR026
+L GND #PWR21
 U 1 1 5AEB80B4
 P 5000 6500
-F 0 "#PWR026" H 5000 6250 50  0001 C CNN
+F 0 "#PWR21" H 5000 6250 50  0001 C CNN
 F 1 "GND" H 5000 6350 50  0000 C CNN
 F 2 "" H 5000 6500 50  0001 C CNN
@@
 	5750 6100 6350 6100
 $Comp
-L GND #PWR027
+L GND #PWR26
 U 1 1 5AEB8909
 P 5800 6850
-F 0 "#PWR027" H 5800 6600 50  0001 C CNN
+F 0 "#PWR26" H 5800 6600 50  0001 C CNN
 F 1 "GND" H 5800 6700 50  0000 C CNN
 F 2 "" H 5800 6850 50  0001 C CNN
@@
 $EndComp
 $Comp
-L GND #PWR028
+L GND #PWR27
 U 1 1 5AEB9284
 P 6050 6400
-F 0 "#PWR028" H 6050 6150 50  0001 C CNN
+F 0 "#PWR27" H 6050 6150 50  0001 C CNN
 F 1 "GND" H 6050 6250 50  0000 C CNN
 F 2 "" H 6050 6400 50  0001 C CNN
@@
 Connection ~ 6050 6100
 $Comp
-L +5V #PWR029
+L +5V #PWR28
 U 1 1 5AEB9666
 P 6350 6000
-F 0 "#PWR029" H 6350 5850 50  0001 C CNN
+F 0 "#PWR28" H 6350 5850 50  0001 C CNN
 F 1 "+5V" H 6350 6140 50  0000 C CNN
 F 2 "" H 6350 6000 50  0001 C CNN
@@
 Connection ~ 5000 5700
 $Comp
-L +12V #PWR030
+L +12V #PWR23
 U 1 1 5AEBA5C2
 P 5200 6050
-F 0 "#PWR030" H 5200 5900 50  0001 C CNN
+F 0 "#PWR23" H 5200 5900 50  0001 C CNN
 F 1 "+12V" H 5200 6190 50  0000 C CNN
 F 2 "" H 5200 6050 50  0001 C CNN
@@
 Connection ~ 5000 6150
 $Comp
-L GND #PWR031
+L GND #PWR25
 U 1 1 5AEBA8BA
 P 5400 6500
-F 0 "#PWR031" H 5400 6250 50  0001 C CNN
+F 0 "#PWR25" H 5400 6250 50  0001 C CNN
 F 1 "GND" H 5400 6350 50  0000 C CNN
 F 2 "" H 5400 6500 50  0001 C CNN
@@
 $EndComp
 $Comp
-L GND #PWR032
+L GND #PWR29
 U 1 1 5AEBAC9B
 P 6350 6400
-F 0 "#PWR032" H 6350 6150 50  0001 C CNN
+F 0 "#PWR29" H 6350 6150 50  0001 C CNN
 F 1 "GND" H 6350 6250 50  0000 C CNN
 F 2 "" H 6350 6400 50  0001 C CNN
@@
 	0    1    1    0
 $EndComp
+$Comp
+L Screw_Terminal_01x02 J5
+U 1 1 5AEC4DA4
+P 1200 5100
+F 0 "J5" H 1200 5200 50  0000 C CNN
+F 1 "12V" H 1200 4900 50  0000 C CNN
+F 2 "" H 1200 5100 50  0001 C CNN
+F 3 "" H 1200 5100 50  0001 C CNN
+	1    1200 5100
+	-1   0    0    1
+$EndComp
+$Comp
+L GND #PWR6
+U 1 1 5AEC4FAE
+P 1400 5100
+F 0 "#PWR6" H 1400 4850 50  0001 C CNN
+F 1 "GND" H 1400 4950 50  0000 C CNN
+F 2 "" H 1400 5100 50  0001 C CNN
+F 3 "" H 1400 5100 50  0001 C CNN
+	1    1400 5100
+	1    0    0    -1
+$EndComp
+$Comp
+L +12V #PWR5
+U 1 1 5AEC51EB
+P 1400 5000
+F 0 "#PWR5" H 1400 4850 50  0001 C CNN
+F 1 "+12V" H 1400 5140 50  0000 C CNN
+F 2 "" H 1400 5000 50  0001 C CNN
+F 3 "" H 1400 5000 50  0001 C CNN
+	1    1400 5000
+	1    0    0    -1
+$EndComp
 $EndSCHEMATC

Commit message: NRF ESP Jumper
Parts:
- removed J1, J2, J3, J4: Conn_01x01, Pin_Headers:Pin_Header_Straight_1x01_Pitch2.54mm, symbol Conn_01x01
- added J1: Conn_02x06_Odd_Even, Pin_Headers:Pin_Header_Straight_2x06_Pitch2.54mm_SMD, symbol Conn_02x06_Odd_Even
- added JP3: Jumper_DeepSleep, LeoDJ-kicad:SOLDER-JUMPER_1-WAY, symbol Jumper_NO_Small
- added JP4, JP5, JP6, JP7, JP8: ESP NRF, LeoDJ-kicad:SOLDER-JUMPER_2-WAY, symbol Jumper_NC_Dual
- added R11: 10k, Resistors_SMD:R_0805_HandSoldering, symbol R
- J5: footprint (none) -> Connectors_Terminal_Blocks:TerminalBlock_Pheonix_MKDS1.5-2pol
- JP1: footprint jumper:SOLDER-JUMPER_2-WAY -> LeoDJ-kicad:SOLDER-JUMPER_2-WAY
- L1: footprint LeoDJ:L_0630 -> LeoDJ-kicad:L_0630
Connections:
- net labels added: ADC, GPIO12, GPIO13, GPIO14, GPIO15, GPIO16, P01, P02, P03, P04, P05, P06, P07, P08, P09, P10, P11, SW
- net labels removed: +VDC
- wire segments 101 -> 133

Commit message: migrate to KiCad5 && further layouting
Parts:
- added C10: 10µF, Capacitor_SMD:C_0805_2012Metric, symbol SHMod24-rescue:C
- added D2: LED, LED_SMD:LED_0805_2012Metric, symbol Device:LED
- added J2, J3: Conn_01x01, Connector_Wire:SolderWirePad_1x01_Drill0.8mm, symbol Connector_Generic:Conn_01x01
- added R12, R13: 10k, Resistor_SMD:R_0805_2012Metric, symbol Device:R
- added R14: 1k, Resistor_SMD:R_0805_2012Metric, symbol Device:R
- added U7: NRF24L01, mysensors_radios:NRF24L01-SMD, symbol SHMod24-rescue:NRF24L01
- C1, C2, C3, C4: footprint Capacitors_SMD:C_0805_HandSoldering -> Capacitor_SMD:C_0805_2012Metric; symbol C -> SHMod24-rescue:C
- C5, C6: footprint Capacitors_SMD:C_0805 -> Capacitor_SMD:C_0805_2012Metric; symbol C -> SHMod24-rescue:C
- C7, C8: footprint Capacitors_SMD:C_1210 -> Capacitor_SMD:C_1210_3225Metric; symbol C -> SHMod24-rescue:C
- C9: footprint Capacitors_SMD:CP_Elec_6.3x5.8 -> Capacitor_SMD:CP_Elec_6.3x5.8; symbol CP -> SHMod24-rescue:CP
- D1: footprint Diodes_SMD:D_SMA -> Diode_SMD:D_SMA; symbol D_Schottky -> SHMod24-rescue:D_Schottky
- IC1: symbol ArduinoProMini -> SHMod24-rescue:ArduinoProMini
- J1: footprint Pin_Headers:Pin_Header_Straight_2x06_Pitch2.54mm_SMD -> Connector_PinHeader_2.54mm:PinHeader_2x06_P2.54mm_Vertical_SMD; symbol Conn_02x06_Odd_Even -> SHMod24-rescue:Conn_02x06_Odd_Even
- J5: footprint Connectors_Terminal_Blocks:TerminalBlock_Pheonix_MKDS1.5-2pol -> TerminalBlock_Phoenix:TerminalBlock_Phoenix_MKDS-1,5-2_1x02_P5.00mm_Horizontal; symbol Screw_Terminal_01x02 -> SHMod24-rescue:Screw_Terminal_01x02
- JP1, JP4, JP5, JP6, JP7, JP8: symbol Jumper_NC_Dual -> SHMod24-rescue:Jumper_NC_Dual
- JP3: symbol Jumper_NO_Small -> SHMod24-rescue:Jumper_NO_Small
- L1: symbol L -> SHMod24-rescue:L
- Q1: footprint Housings_SSOP:TSSOP-8_4.4x3mm_Pitch0.65mm -> Package_SO:TSSOP-8_4.4x3mm_P0.65mm; symbol FS8205A -> SHMod24-rescue:FS8205A
- R1, R11, R2, R3, R4, R5, R6, R7, R8: footprint Resistors_SMD:R_0805_HandSoldering -> Resistor_SMD:R_0805_2012Metric; symbol R -> SHMod24-rescue:R
- R10, R9: footprint Resistors_SMD:R_0805 -> Resistor_SMD:R_0805_2012Metric; symbol R -> SHMod24-rescue:R
- U1: symbol ESP-12 -> SHMod24-rescue:ESP-12
- U2: symbol NRF24L01 -> SHMod24-rescue:NRF24L01
- U3: footprint TO_SOT_Packages_SMD:SOT-23-5 -> Package_TO_SOT_SMD:SOT-23-5; symbol AP2204K-3.3 -> SHMod24-rescue:AP2204K-3.3
- U4: footprint Housings_SOIC:SOIC-8_3.9x4.9mm_Pitch1.27mm -> Package_SO:SOIC-8_3.9x4.9mm_P1.27mm; symbol TP4056 -> SHMod24-rescue:TP4056
- U5: footprint TO_SOT_Packages_SMD:SOT-23-6_Handsoldering -> Package_TO_SOT_SMD:SOT-23-6_Handsoldering; symbol DW01A -> SHMod24-rescue:DW01A
- U6: footprint TO_SOT_Packages_SMD:SOT-23-6_Handsoldering -> Package_TO_SOT_SMD:SOT-23-6_Handsoldering; symbol LMR14010A -> SHMod24-rescue:LMR14010A
Connections:
- net labels added: VCC
- net labels removed: +12V
- wire segments 133 -> 159

Commit message: more layouting
Parts:
- removed J1: Conn_02x06_Odd_Even, Connector_PinHeader_2.54mm:PinHeader_2x06_P2.54mm_Vertical_SMD, symbol SHMod24-rescue:Conn_02x06_Odd_Even
- added J?: Conn_02x14_Odd_Even, symbol Connector_Generic:Conn_02x14_Odd_Even
Connections:
- net labels added: A1, A2, A3, CS
- net labels removed: P01, P08, P11
- wire segments 159 -> 147

Commit message: even more layouting
Parts:
- J1: renamed from J?; footprint (none) -> Connector_PinHeader_2.54mm:PinHeader_2x14_P2.54mm_Vertical_SMD
Changed lines of the file:
@@
 	2300 7100 2300 7250
 $Comp
-L power:GND #PWR?
+L power:GND #PWR0111
 U 1 1 5B043100
 P 1100 4950
-F 0 "#PWR?" H 1100 4700 50  0001 C CNN
+F 0 "#PWR0111" H 1100 4700 50  0001 C CNN
 F 1 "GND" H 1105 4777 50  0000 C CNN
 F 2 "" H 1100 4950 50  0001 C CNN
@@
 $EndComp
 $Comp
-L power:GND #PWR?
+L power:GND #PWR0112
 U 1 1 5B043170
 P 950 4250
-F 0 "#PWR?" H 950 4000 50  0001 C CNN
+F 0 "#PWR0112" H 950 4000 50  0001 C CNN
 F 1 "GND" H 955 4077 50  0000 C CNN
 F 2 "" H 950 4250 50  0001 C CNN
@@
 	1100 4250 1100 4450
 $Comp
-L power:+3V3 #PWR?
+L power:+3V3 #PWR0113
 U 1 1 5B0690C4
 P 1300 4450
-F 0 "#PWR?" H 1300 4300 50  0001 C CNN
+F 0 "#PWR0113" H 1300 4300 50  0001 C CNN
 F 1 "+3V3" H 1315 4623 50  0000 C CNN
 F 2 "" H 1300 4450 50  0001 C CNN
@@
 $EndComp
 $Comp
-L power:+3V3 #PWR?
+L power:+3V3 #PWR0114
 U 1 1 5B069134
 P 1350 5400
-F 0 "#PWR?" H 1350 5250 50  0001 C CNN
+F 0 "#PWR0114" H 1350 5250 50  0001 C CNN
 F 1 "+3V3" H 1365 5573 50  0000 C CNN
 F 2 "" H 1350 5400 50  0001 C CNN
@@
 $EndComp
 $Comp
-L power:+5V #PWR?
+L power:+5V #PWR0115
 U 1 1 5B0693A1
 P 1150 5400
-F 0 "#PWR?" H 1150 5250 50  0001 C CNN
+F 0 "#PWR0115" H 1150 5250 50  0001 C CNN
 F 1 "+5V" H 1165 5573 50  0000 C CNN
 F 2 "" H 1150 5400 50  0001 C CNN
@@
 $EndComp
 $Comp
-L power:VCC #PWR?
+L power:VCC #PWR0116
 U 1 1 5B06944B
 P 1200 4350
-F 0 "#PWR?" H 1200 4200 50  0001 C CNN
+F 0 "#PWR0116" H 1200 4200 50  0001 C CNN
 F 1 "VCC" H 1217 4523 50  0000 C CNN
 F 2 "" H 1200 4350 50  0001 C CNN
@@
 GPIO2
 $Comp
-L power:GND #PWR?
+L power:GND #PWR0117
 U 1 1 5B199E3F
 P 2000 4950
-F 0 "#PWR?" H 2000 4700 50  0001 C CNN
+F 0 "#PWR0117" H 2000 4700 50  0001 C CNN
 F 1 "GND" H 2005 4777 50  0000 C CNN
 F 2 "" H 2000 4950 50  0001 C CNN
@@
 $EndComp
 $Comp
-L power:GND #PWR?
+L power:GND #PWR0118
 U 1 1 5B199EA8
 P 1900 4100
-F 0 "#PWR?" H 1900 3850 50  0001 C CNN
+F 0 "#PWR0118" H 1900 3850 50  0001 C CNN
 F 1 "GND" H 1905 3927 50  0000 C CNN
 F 2 "" H 1900 4100 50  0001 C CNN
@@
 	2000 4100 2000 4450
 $Comp
-L Connector_Generic:Conn_02x14_Odd_Even J?
+L Connector_Generic:Conn_02x14_Odd_Even J1
 U 1 1 5B1A025A
 P 1700 4750
-F 0 "J?" V 1796 3962 50  0000 R CNN
+F 0 "J1" V 1796 3962 50  0000 R CNN
 F 1 "Conn_02x14_Odd_Even" V 1705 3962 50  0000 R CNN
-F 2 "" H 1700 4750 50  0001 C CNN
+F 2 "Connector_PinHeader_2.54mm:PinHeader_2x14_P2.54mm_Vertical_SMD" H 1700 4750 50  0001 C CNN
 F 3 "~" H 1700 4750 50  0001 C CNN
 	1    1700 4750

Commit message: layouting of the current schematic complete
Parts:
- removed JP4, JP5, JP6, JP7, JP8: ESP NRF, LeoDJ-kicad:SOLDER-JUMPER_2-WAY, symbol SHMod24-rescue:Jumper_NC_Dual
- D2: symbol Device:LED -> SHMod24-rescue:LED-Device
- J1: symbol Connector_Generic:Conn_02x14_Odd_Even -> SHMod24-rescue:Conn_02x14_Odd_Even-Connector_Generic
- J2, J3: symbol Connector_Generic:Conn_01x01 -> SHMod24-rescue:Conn_01x01-Connector_Generic
- R12, R13, R14: symbol Device:R -> SHMod24-rescue:R-Device
Connections:
- wire segments 147 -> 136
Changed lines of the file:
@@
 Text Label 5000 6600 0    20   ~ 0
 SW
-$Comp
-L SHMod24-rescue:Jumper_NC_Dual JP8
-U 1 1 5AEC6742
-P 3950 2950
-F 0 "JP8" H 4000 2850 50  0000 L CNN
-F 1 "ESP NRF" H 3950 3050 50  0000 C BNN
-F 2 "LeoDJ-kicad:SOLDER-JUMPER_2-WAY" H 3950 2950 50  0001 C CNN
-F 3 "" H 3950 2950 50  0001 C CNN
-	1    3950 2950
-	1    0    0    -1
-$EndComp
 Text GLabel 4100 2300 2    60   BiDi ~ 0
 GPIO15
@@
 Text GLabel 2900 3350 0    60   BiDi ~ 0
 GPIO15
-Wire Wire Line
-	3950 3050 3700 3050
-Wire Wire Line
-	3700 3050 3700 2950
-Text GLabel 2900 3350 2    60   BiDi ~ 0
+Text GLabel 2950 3350 2    60   BiDi ~ 0
 N24_CS
-Wire Wire Line
-	3900 3150 3950 3150
-Wire Wire Line
-	3950 3150 3950 3050
 Text GLabel 2400 4950 3    47   BiDi ~ 0
 P10
@@
 Text GLabel 2300 4950 3    47   BiDi ~ 0
 P07
-$Comp
-L SHMod24-rescue:Jumper_NC_Dual JP4
-U 1 1 5AECA1CD
-P 3950 3400
-F 0 "JP4" H 4000 3300 50  0000 L CNN
-F 1 "ESP NRF" H 3950 3500 50  0000 C BNN
-F 2 "LeoDJ-kicad:SOLDER-JUMPER_2-WAY" H 3950 3400 50  0001 C CNN
-F 3 "" H 3950 3400 50  0001 C CNN
-	1    3950 3400
-	1    0    0    -1
-$EndComp
-Wire Wire Line
-	3950 3500 3700 3500
-Wire Wire Line
-	3700 3500 3700 3400
-Wire Wire Line
-	3950 3600 3950 3500
-$Comp
-L SHMod24-rescue:Jumper_NC_Dual JP5
-U 1 1 5AECA2AF
-P 3950 3900
-F 0 "JP5" H 4000 3800 50  0000 L CNN
-F 1 "ESP NRF" H 3950 4000 50  0000 C BNN
-F 2 "LeoDJ-kicad:SOLDER-JUMPER_2-WAY" H 3950 3900 50  0001 C CNN
-F 3 "" H 3950 3900 50  0001 C CNN
-	1    3950 3900
-	1    0    0    -1
-$EndComp
-Wire Wire Line
-	3950 4000 3700 4000
-Wire Wire Line
-	3700 4000 3700 3900
-Wire Wire Line
-	3950 4100 3950 4000
-$Comp
-L SHMod24-rescue:Jumper_NC_Dual JP6
-U 1 1 5AECA44E
-P 3950 4400
-F 0 "JP6" H 4000 4300 50  0000 L CNN
-F 1 "ESP NRF" H 3950 4500 50  0000 C BNN
-F 2 "LeoDJ-kicad:SOLDER-JUMPER_2-WAY" H 3950 4400 50  0001 C CNN
-F 3 "" H 3950 4400 50  0001 C CNN
-	1    3950 4400
-	1    0    0    -1
-$EndComp
-Wire Wire Line
-	3950 4500 3700 4500
-Wire Wire Line
-	3700 4500 3700 4400
-Wire Wire Line
-	3950 4600 3950 4500
-$Comp
-L SHMod24-rescue:Jumper_NC_Dual JP7
-U 1 1 5AECA457
-P 3950 4900
-F 0 "JP7" H 4000 4800 50  0000 L CNN
-F 1 "ESP NRF" H 3950 5000 50  0000 C BNN
-F 2 "LeoDJ-kicad:SOLDER-JUMPER_2-WAY" H 3950 4900 50  0001 C CNN
-F 3 "" H 3950 4900 50  0001 C CNN
-	1    3950 4900
-	1    0    0    -1
-$EndComp
-Wire Wire Line
-	3950 5000 3700 5000
-Wire Wire Line
-	3700 5000 3700 4900
-Wire Wire Line
-	3950 5100 3950 5000
 Text GLabel 2050 2300 0    60   BiDi ~ 0
 GPIO13
@@
 Text GLabel 2900 3450 0    60   BiDi ~ 0
 GPIO13
-Wire Wire Line
-	3950 3600 3900 3600
 Text GLabel 2900 3550 0    60   BiDi ~ 0
 GPIO12
@@
 Wire Wire Line
 	1050 2500 1100 2500
-Text GLabel 2900 3450 2    60   BiDi ~ 0
+Text GLabel 2950 3450 2    60   BiDi ~ 0
 MOSI
-Text GLabel 2900 3550 2    60   BiDi ~ 0
+Text GLabel 2950 3550 2    60   BiDi ~ 0
 MISO
-Text GLabel 2900 3650 2    60   BiDi ~ 0
+Text GLabel 2950 3650 2    60   BiDi ~ 0
 SCK
-Text GLabel 2900 3250 2    60   BiDi ~ 0
+Text GLabel 2950 3250 2    60   BiDi ~ 0
 N24_CE
 Text GLabel 2900 3250 0    60   BiDi ~ 0
 GPIO16
-Wire Wire Line
-	3950 4100 3900 4100
-Wire Wire Line
-	3950 4600 3900 4600
-Wire Wire Line
-	3900 5100 3950 5100
 Wire Wire Line
 	5200 3000 5200 3200
@@
 $EndComp
 $Comp
-L power:+BATT #PWR0103
+L SHMod24-rescue:+BATT-power #PWR0103
 U 1 1 5B02FB2C
 P 1700 3200
@@
 $EndComp
 $Comp
-L power:-BATT #PWR0104
+L SHMod24-rescue:-BATT-power #PWR0104
 U 1 1 5B02FC02
 P 1700 3300
@@
 $EndComp
 $Comp
-L Connector_Generic:Conn_01x01 J2
+L SHMod24-rescue:Conn_01x01-Connector_Generic J2
 U 1 1 5B0307B4
 P 1500 3200
@@
 $EndComp
 $Comp
-L Connector_Generic:Conn_01x01 J3
+L SHMod24-rescue:Conn_01x01-Connector_Generic J3
 U 1 1 5B030925
 P 1500 3300
@@
 	10650 3000 10550 3000
 $Comp
-L power:+3V3 #PWR0107
+L SHMod24-rescue:+3V3-power #PWR0107
 U 1 1 5B04FE9B
 P 4000 900
@@
 $EndComp
 $Comp
-L Device:R R12
+L SHMod24-rescue:R-Device R12
 U 1 1 5B05001C
 P 4000 1050
@@
 $EndComp
 $Comp
-L Device:R R13
+L SHMod24-rescue:R-Device R13
 U 1 1 5B050098
 P 4250 1050
@@
 $EndComp
 $Comp
-L power:+3V3 #PWR0108
+L SHMod24-rescue:+3V3-power #PWR0108
 U 1 1 5B066B95
 P 4250 900
@@
 SCL
 $Comp
-L power:VCC #PWR0109
+L SHMod24-rescue:VCC-power #PWR0109
 U 1 1 5B0778C1
 P 5200 6700
@@
 $EndComp
 $Comp
-L power:VCC #PWR0110
+L SHMod24-rescue:VCC-power #PWR0110
 U 1 1 5B077B87
 P 1050 3200
@@
 $EndComp
 $Comp
-L Device:R R14
+L SHMod24-rescue:R-Device R14
 U 1 1 5B07F902
 P 2150 6800
@@
 $EndComp
 $Comp
-L Device:LED D2
+L SHMod24-rescue:LED-Device D2
 U 1 1 5B07F9BB
 P 2300 6950
@@
 	2300 7100 2300 7250
 $Comp
-L power:GND #PWR0111
+L SHMod24-rescue:GND-power #PWR0111
 U 1 1 5B043100
 P 1100 4950
@@
 $EndComp
 $Comp
-L power:GND #PWR0112
+L SHMod24-rescue:GND-power #PWR0112
 U 1 1 5B043170
 P 950 4250
@@
 	1100 4250 1100 4450
 $Comp
-L power:+3V3 #PWR0113
+L SHMod24-rescue:+3V3-power #PWR0113
 U 1 1 5B0690C4
 P 1300 4450
@@
 $EndComp
 $Comp
-L power:+3V3 #PWR0114
+L SHMod24-rescue:+3V3-power #PWR0114
 U 1 1 5B069134
 P 1350 5400
@@
 $EndComp
 $Comp
-L power:+5V #PWR0115
+L SHMod24-rescue:+5V-power #PWR0115
 U 1 1 5B0693A1
 P 1150 5400
@@
 $EndComp
 $Comp
-L power:VCC #PWR0116
+L SHMod24-rescue:VCC-power #PWR0116
 U 1 1 5B06944B
 P 1200 4350
@@
 Text GLabel 7150 2600 2    60   BiDi ~ 0
 A3
-Text GLabel 3200 4600 2    47   BiDi ~ 0
+Text GLabel 3250 4600 2    47   BiDi ~ 0
 CS
 Text GLabel 1700 4950 3    47   BiDi ~ 0
@@
 Text GLabel 7150 900  2    60   BiDi ~ 0
 P02
-Text GLabel 3200 4500 2    47   BiDi ~ 0
+Text GLabel 3250 4500 2    47   BiDi ~ 0
 P07
-Text GLabel 2900 3800 2    47   BiDi ~ 0
+Text GLabel 2950 3800 2    47   BiDi ~ 0
 P02
-Text GLabel 2900 3900 2    47   BiDi ~ 0
+Text GLabel 2950 3900 2    47   BiDi ~ 0
 P03
 Text GLabel 2900 3800 0    47   BiDi ~ 0
@@
 GPIO2
 $Comp
-L power:GND #PWR0117
+L SHMod24-rescue:GND-power #PWR0117
 U 1 1 5B199E3F
 P 2000 4950
@@
 $EndComp
 $Comp
-L power:GND #PWR0118
+L SHMod24-rescue:GND-power #PWR0118
 U 1 1 5B199EA8
 P 1900 4100
@@
 	2000 4100 2000 4450
 $Comp
-L Connector_Generic:Conn_02x14_Odd_Even J1
+L SHMod24-rescue:Conn_02x14_Odd_Even-Connector_Generic J1
 U 1 1 5B1A025A
 P 1700 4750
@@
 	0    -1   -1   0
 $EndComp
+Wire Wire Line
+	2950 3250 2900 3250
+Wire Wire Line
+	2950 3350 2900 3350
+Wire Wire Line
+	2950 3450 2900 3450
+Wire Wire Line
+	2950 3550 2900 3550
+Wire Wire Line
+	2950 3650 2900 3650
+Wire Wire Line
+	2950 3800 2900 3800
+Wire Wire Line
+	2950 3900 2900 3900
+Wire Wire Line
+	3250 4500 3200 4500
+Wire Wire Line
+	3250 4600 3200 4600
 $EndSCHEMATC
