File: SHMod24.sch (KiCad schematic (older format))
At the start: 54 parts, among them IC1 ArduinoProMini, J1 Conn_02x14_Odd_Even, J2 Conn_01x01, J3 Conn_01x01, J4 RESET, J5 12V, J6 GND, J9 Screw_Terminal_01x02, Q1 FS8205A, Q2 AO3400A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

Commit message: add MOSFET pulldowns
Parts:
- added R16, R17, R18, R19: 10k, Resistor_SMD:R_0603_1608Metric, symbol Device:R
Connections:
- wire segments 158 -> 170
Changed lines of the file:
@@
 Text GLabel 5950 4350 0    47   BiDi ~ 0
 P05
+$Comp
+L Device:R R16
+U 1 1 5B1BFF57
+P 4850 4500
+F 0 "R16" H 4780 4454 50  0000 R CNN
+F 1 "10k" H 4780 4545 50  0000 R CNN
+F 2 "Resistor_SMD:R_0603_1608Metric" V 4780 4500 50  0001 C CNN
+F 3 "~" H 4850 4500 50  0001 C CNN
+	1    4850 4500
+	-1   0    0    1
+$EndComp
+Connection ~ 4850 4350
+$Comp
+L Device:R R18
+U 1 1 5B1C00EF
+P 5950 4500
+F 0 "R18" H 5880 4454 50  0000 R CNN
+F 1 "10k" H 5880 4545 50  0000 R CNN
+F 2 "Resistor_SMD:R_0603_1608Metric" V 5880 4500 50  0001 C CNN
+F 3 "~" H 5950 4500 50  0001 C CNN
+	1    5950 4500
+	-1   0    0    1
+$EndComp
+Connection ~ 5950 4350
+$Comp
+L Device:R R19
+U 1 1 5B1C0199
+P 5950 5150
+F 0 "R19" H 5880 5104 50  0000 R CNN
+F 1 "10k" H 5880 5195 50  0000 R CNN
+F 2 "Resistor_SMD:R_0603_1608Metric" V 5880 5150 50  0001 C CNN
+F 3 "~" H 5950 5150 50  0001 C CNN
+	1    5950 5150
+	-1   0    0    1
+$EndComp
+Connection ~ 5950 5000
+$Comp
+L Device:R R17
+U 1 1 5B1C0237
+P 4850 5150
+F 0 "R17" H 4780 5104 50  0000 R CNN
+F 1 "10k" H 4780 5195 50  0000 R CNN
+F 2 "Resistor_SMD:R_0603_1608Metric" V 4780 5150 50  0001 C CNN
+F 3 "~" H 4850 5150 50  0001 C CNN
+	1    4850 5150
+	-1   0    0    1
+$EndComp
+Connection ~ 4850 5000
+Wire Wire Line
+	4850 4650 5100 4650
+Wire Wire Line
+	5100 4650 5100 4550
+Wire Wire Line
+	5100 4550 5150 4550
+Connection ~ 5150 4550
+Wire Wire Line
+	5950 4650 6200 4650
+Wire Wire Line
+	6200 4650 6200 4550
+Wire Wire Line
+	6200 4550 6250 4550
+Connection ~ 6250 4550
+Wire Wire Line
+	4850 5300 5100 5300
+Wire Wire Line
+	5100 5300 5100 5200
+Wire Wire Line
+	5100 5200 5150 5200
+Connection ~ 5150 5200
+Wire Wire Line
+	5950 5300 6200 5300
+Wire Wire Line
+	6200 5300 6200 5200
+Wire Wire Line
+	6200 5200 6250 5200
+Connection ~ 6250 5200
 $EndSCHEMATC

Commit message: add fifth MOSFET
Parts:
- added Q6: AO3400A, Package_TO_SOT_SMD:SOT-23, symbol LeoDJ-kicad:AO3400A
- added R20: 10k, Resistor_SMD:R_0603_1608Metric, symbol Device:R
Connections:
- wire segments 170 -> 175
Changed lines of the file:
@@
 	6200 5200 6250 5200
 Connection ~ 6250 5200
+Text GLabel 3850 4350 0    47   BiDi ~ 0
+P03
+$Comp
+L LeoDJ-kicad:AO3400A Q6
+U 1 1 5B1DF661
+P 4050 4350
+F 0 "Q6" H 4256 4396 50  0000 L CNN
+F 1 "AO3400A" H 4256 4305 50  0000 L CNN
+F 2 "Package_TO_SOT_SMD:SOT-23" H 4250 4275 50  0001 L CIN
+F 3 "http://www.aosmd.com/pdfs/datasheet/AO3400A.pdf" H 4050 4350 50  0001 L CNN
+	1    4050 4350
+	1    0    0    -1
+$EndComp
+Wire Wire Line
+	4150 4150 3850 4150
+Wire Wire Line
+	3850 4150 3850 4350
+$Comp
+L power:GND #PWR0126
+U 1 1 5B1DF66B
+P 4150 4550
+F 0 "#PWR0126" H 4150 4300 50  0001 C CNN
+F 1 "GND" H 4155 4377 50  0000 C CNN
+F 2 "" H 4150 4550 50  0001 C CNN
+F 3 "" H 4150 4550 50  0001 C CNN
+	1    4150 4550
+	1    0    0    -1
+$EndComp
+$Comp
+L Device:R R20
+U 1 1 5B1DF671
+P 3850 4500
+F 0 "R20" H 3780 4454 50  0000 R CNN
+F 1 "10k" H 3780 4545 50  0000 R CNN
+F 2 "Resistor_SMD:R_0603_1608Metric" V 3780 4500 50  0001 C CNN
+F 3 "~" H 3850 4500 50  0001 C CNN
+	1    3850 4500
+	-1   0    0    1
+$EndComp
+Connection ~ 3850 4350
+Wire Wire Line
+	3850 4650 4100 4650
+Wire Wire Line
+	4100 4650 4100 4550
+Wire Wire Line
+	4100 4550 4150 4550
+Connection ~ 4150 4550
 $EndSCHEMATC

Commit message: add high voltage sense input
Parts:
- added JP2: VoltSense, LeoDJ-kicad:SOLDER-JUMPER_2-WAY, symbol SHMod24-rescue:Jumper_NC_Dual
- added R21: 47k/220k, Resistor_SMD:R_0805_2012Metric, symbol Device:R
- added R22: 22k, Resistor_SMD:R_0805_2012Metric, symbol Device:R
Connections:
- wire segments 175 -> 180

Commit message: begin switching regulator improvement
Changed lines of the file:
@@
 	1    0    0    -1
 $EndComp
-Wire Wire Line
-	5000 6700 5000 6800
 $Comp
 L SHMod24-rescue:GND #PWR021
@@
 L SHMod24-rescue:C C7
 U 1 1 5AEB7F2F
-P 5000 6950
-F 0 "C7" H 4900 7050 50  0000 L CNN
-F 1 "2.2µF 50V" H 4750 6850 50  0000 L CNN
-F 2 "Capacitor_SMD:C_1210_3225Metric" H 5038 6800 50  0001 C CNN
-F 3 "" H 5000 6950 50  0001 C CNN
-	1    5000 6950
+P 5100 6850
+F 0 "C7" H 5000 6950 50  0000 L CNN
+F 1 "2.2µF 50V" H 4850 6750 50  0000 L CNN
+F 2 "Capacitor_SMD:C_1210_3225Metric" H 5138 6700 50  0001 C CNN
+F 3 "" H 5100 6850 50  0001 C CNN
+	1    5100 6850
 	1    0    0    -1
 $EndComp
@@
 L SHMod24-rescue:GND #PWR022
 U 1 1 5AEB80B4
-P 5000 7150
-F 0 "#PWR022" H 5000 6900 50  0001 C CNN
-F 1 "GND" H 5000 7000 50  0000 C CNN
-F 2 "" H 5000 7150 50  0001 C CNN
-F 3 "" H 5000 7150 50  0001 C CNN
-	1    5000 7150
+P 5100 7050
+F 0 "#PWR022" H 5100 6800 50  0001 C CNN
+F 1 "GND" H 5100 6900 50  0000 C CNN
+F 2 "" H 5100 7050 50  0001 C CNN
+F 3 "" H 5100 7050 50  0001 C CNN
+	1    5100 7050
 	1    0    0    -1
 $EndComp
@@
 	4750 6350 5000 6350
 Wire Wire Line
-	5000 7150 5000 7100
+	5100 7050 5100 7000
 Wire Wire Line
 	5400 6350 5400 6750
@@
 Connection ~ 5000 6350
 Wire Wire Line
-	5200 6700 5000 6700
-Connection ~ 5000 6700
-Connection ~ 5000 6800
+	5200 6700 5100 6700
 $Comp
 L SHMod24-rescue:GND #PWR027
@@
 	4350 3400 4150 3400
 Connection ~ 4150 3400
+Connection ~ 5100 6700
+Wire Wire Line
+	5100 6700 5000 6700
 $EndSCHEMATC

Commit message: add power LED && place references better
Parts:
- added D3: LED, LED_SMD:LED_0805_2012Metric, symbol Device:LED
- added R23: 1k, Resistor_SMD:R_0805_2012Metric, symbol Device:R
Changed lines of the file:
@@
 Wire Wire Line
 	5100 6700 5000 6700
+$Comp
+L Device:R R23
+U 1 1 5B26AF85
+P 4700 4050
+F 0 "R23" H 4770 4096 50  0000 L CNN
+F 1 "1k" H 4770 4005 50  0000 L CNN
+F 2 "Resistor_SMD:R_0805_2012Metric" V 4630 4050 50  0001 C CNN
+F 3 "~" H 4700 4050 50  0001 C CNN
+	1    4700 4050
+	1    0    0    -1
+$EndComp
+$Comp
+L Device:LED D3
+U 1 1 5B26B071
+P 4700 4350
+F 0 "D3" V 4738 4233 50  0000 R CNN
+F 1 "LED" V 4647 4233 50  0000 R CNN
+F 2 "LED_SMD:LED_0805_2012Metric" H 4700 4350 50  0001 C CNN
+F 3 "~" H 4700 4350 50  0001 C CNN
+	1    4700 4350
+	0    -1   -1   0
+$EndComp
+$Comp
+L power:+3.3V #PWR0130
+U 1 1 5B26B1FA
+P 4700 3900
+F 0 "#PWR0130" H 4700 3750 50  0001 C CNN
+F 1 "+3.3V" H 4715 4073 50  0000 C CNN
+F 2 "" H 4700 3900 50  0001 C CNN
+F 3 "" H 4700 3900 50  0001 C CNN
+	1    4700 3900
+	1    0    0    -1
+$EndComp
+$Comp
+L power:GND #PWR0131
+U 1 1 5B26B2B3
+P 4700 4500
+F 0 "#PWR0131" H 4700 4250 50  0001 C CNN
+F 1 "GND" H 4705 4327 50  0000 C CNN
+F 2 "" H 4700 4500 50  0001 C CNN
+F 3 "" H 4700 4500 50  0001 C CNN
+	1    4700 4500
+	1    0    0    -1
+$EndComp
 $EndSCHEMATC

Commit message: fix LDO no GND && minor trace improvements
Parts:
- added C11: 100n, Capacitor_SMD:C_0805_2012Metric, symbol SHMod24-rescue:C
- R6: value 1k2 -> 2k2
Connections:
- wire segments 180 -> 182
Changed lines of the file:
@@
 P 650 7400
 F 0 "R6" V 730 7400 50  0000 C CNN
-F 1 "1k2" V 650 7400 50  0000 C CNN
+F 1 "2k2" V 650 7400 50  0000 C CNN
 F 2 "Resistor_SMD:R_0805_2012Metric" V 580 7400 50  0001 C CNN
 F 3 "" H 650 7400 50  0001 C CNN
@@
 	1    0    0    -1
 $EndComp
+$Comp
+L power:GND #PWR0132
+U 1 1 5B28B10B
+P 9850 5850
+F 0 "#PWR0132" H 9850 5600 50  0001 C CNN
+F 1 "GND" H 9855 5677 50  0000 C CNN
+F 2 "" H 9850 5850 50  0001 C CNN
+F 3 "" H 9850 5850 50  0001 C CNN
+	1    9850 5850
+	1    0    0    -1
+$EndComp
+$Comp
+L SHMod24-rescue:C C11
+U 1 1 5B28F72B
+P 9400 850
+F 0 "C11" H 9425 950 50  0000 L CNN
+F 1 "100n" H 9425 750 50  0000 L CNN
+F 2 "Capacitor_SMD:C_0805_2012Metric" H 9438 700 50  0001 C CNN
+F 3 "" H 9400 850 50  0001 C CNN
+	1    9400 850
+	1    0    0    -1
+$EndComp
+Wire Wire Line
+	9400 1000 9650 1000
+Connection ~ 9650 1000
+Wire Wire Line
+	9400 700  9650 700
+Connection ~ 9650 700
 $EndSCHEMATC

Commit message: more layout improvements
Parts:
- added JP4, JP5: ESP_MOSFET, LeoDJ-kicad:SOLDER-JUMPER_1-WAY, symbol SHMod24-rescue:Jumper_NO_Small
Connections:
- wire segments 182 -> 180
Changed lines of the file:
@@
 	10150 1850 10150 1700
 Wire Wire Line
-	5200 3000 5250 3000
-Wire Wire Line
 	5200 2800 5200 2900
 Wire Wire Line
 	5250 2900 5200 2900
-Connection ~ 5200 3000
 Wire Wire Line
 	5250 2800 5200 2800
@@
 Text GLabel 3000 3450 0    60   BiDi ~ 0
 GPIO16
-Wire Wire Line
-	5200 3000 5200 3200
-Wire Wire Line
-	5200 2900 5200 3000
 Wire Wire Line
 	650  1900 650  2100
@@
 	9400 700  9650 700
 Connection ~ 9650 700
+Wire Wire Line
+	5200 2900 5200 3200
+$Comp
+L SHMod24-rescue:Jumper_NO_Small JP4
+U 1 1 5B3023D8
+P 4100 4900
+F 0 "JP4" H 4100 4980 50  0000 C CNN
+F 1 "ESP_MOSFET" H 4110 4840 50  0000 C CNN
+F 2 "LeoDJ-kicad:SOLDER-JUMPER_1-WAY" H 4100 4900 50  0001 C CNN
+F 3 "" H 4100 4900 50  0001 C CNN
+	1    4100 4900
+	-1   0    0    1
+$EndComp
+$Comp
+L SHMod24-rescue:Jumper_NO_Small JP5
+U 1 1 5B3026D2
+P 4100 5150
+F 0 "JP5" H 4100 5230 50  0000 C CNN
+F 1 "ESP_MOSFET" H 4110 5090 50  0000 C CNN
+F 2 "LeoDJ-kicad:SOLDER-JUMPER_1-WAY" H 4100 5150 50  0001 C CNN
+F 3 "" H 4100 5150 50  0001 C CNN
+	1    4100 5150
+	-1   0    0    1
+$EndComp
+Text GLabel 4200 4900 2    47   BiDi ~ 0
+P05
+Text GLabel 4200 5150 2    47   BiDi ~ 0
+P06
+Text GLabel 4000 4900 0    60   BiDi ~ 0
+GPIO13
+Text GLabel 4000 5150 0    60   BiDi ~ 0
+GPIO12
 $EndSCHEMATC

Commit message: more improvements
Parts:
- added R24: 10k, Resistor_SMD:R_0805_2012Metric, symbol SHMod24-rescue:R
Connections:
- wire segments 180 -> 183
Other:
- note added: "MOSFETs can be optionally fitted\nFor that the trace bridging gate and source has to be cut\nIn the layout this is implemented manually"
