File: SHMod24.sch (KiCad schematic (older format))
At the start: 69 parts, among them IC1 ArduinoProMini, J1 Conn_02x14_Odd_Even, J2 Conn_01x01, J3 Conn_01x01, J4 RESET, J5 12V, J6 GND, J9 Screw_Terminal_01x02, Q1 FS8205A, Q2 AO3400A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

Commit message: final improvements: better track layout, silk screen symbols
Parts:
- added LOGO1: Logo_Open_Hardware_Small, Symbol:OSHW-Logo2_7.3x6mm_SilkScreen, symbol Graphic:Logo_Open_Hardware_Small
- added SYM1: SYM_Arrow_Tiny, leodj-kicad:Otter_Lightbulb_smaller, symbol Graphic:SYM_Arrow_Tiny
- added SYM2: SYM_Arrow_Tiny, leodj-kicad:QR_Code_SHMod24, symbol Graphic:SYM_Arrow_Tiny
- C1, C10, C11, C2, C3, C4, C5, C6: footprint Capacitor_SMD:C_0805_2012Metric -> LeoDJ-kicad:C_0805_2012Metric
- R1, R10, R11, R12, R13, R14, R15, R2, R21, R22, R23, R24, R3, R4, R5, R6, R7, R8, R9: footprint Resistor_SMD:R_0805_2012Metric -> LeoDJ-kicad:R_0805_2012Metric
Other:
- note added: "^ Logos"
Changed lines of the file:
@@
 F 0 "R1" V 980 1900 50  0000 C CNN
 F 1 "10k" V 900 1900 50  0000 C CNN
-F 2 "Resistor_SMD:R_0805_2012Metric" V 830 1900 50  0001 C CNN
+F 2 "LeoDJ-kicad:R_0805_2012Metric" V 830 1900 50  0001 C CNN
 F 3 "" H 900 1900 50  0001 C CNN
 	1    900  1900
@@
 F 0 "R2" V 980 2100 50  0000 C CNN
 F 1 "10k" V 900 2100 50  0000 C CNN
-F 2 "Resistor_SMD:R_0805_2012Metric" V 830 2100 50  0001 C CNN
+F 2 "LeoDJ-kicad:R_0805_2012Metric" V 830 2100 50  0001 C CNN
 F 3 "" H 900 2100 50  0001 C CNN
 	1    900  2100
@@
 F 0 "R3" V 980 2300 50  0000 C CNN
 F 1 "10k" V 900 2300 50  0000 C CNN
-F 2 "Resistor_SMD:R_0805_2012Metric" V 830 2300 50  0001 C CNN
+F 2 "LeoDJ-kicad:R_0805_2012Metric" V 830 2300 50  0001 C CNN
 F 3 "" H 900 2300 50  0001 C CNN
 	1    900  2300
@@
 F 0 "R5" V 1580 1150 50  0000 C CNN
 F 1 "100k" V 1500 1150 50  0000 C CNN
-F 2 "Resistor_SMD:R_0805_2012Metric" V 1430 1150 50  0001 C CNN
+F 2 "LeoDJ-kicad:R_0805_2012Metric" V 1430 1150 50  0001 C CNN
 F 3 "" H 1500 1150 50  0001 C CNN
 	1    1500 1150
@@
 F 0 "R4" V 1580 750 50  0000 C CNN
 F 1 "220k" V 1500 750 50  0000 C CNN
-F 2 "Resistor_SMD:R_0805_2012Metric" V 1430 750 50  0001 C CNN
+F 2 "LeoDJ-kicad:R_0805_2012Metric" V 1430 750 50  0001 C CNN
 F 3 "" H 1500 750 50  0001 C CNN
 	1    1500 750
@@
 F 0 "C1" H 9125 5700 50  0000 L CNN
 F 1 "1µF" H 9125 5500 50  0000 L CNN
-F 2 "Capacitor_SMD:C_0805_2012Metric" H 9138 5450 50  0001 C CNN
+F 2 "LeoDJ-kicad:C_0805_2012Metric" H 9138 5450 50  0001 C CNN
 F 3 "" H 9100 5600 50  0001 C CNN
 	1    9100 5600
@@
 F 0 "C2" H 10425 5700 50  0000 L CNN
 F 1 "1µF" H 10425 5500 50  0000 L CNN
-F 2 "Capacitor_SMD:C_0805_2012Metric" H 10438 5450 50  0001 C CNN
+F 2 "LeoDJ-kicad:C_0805_2012Metric" H 10438 5450 50  0001 C CNN
 F 3 "" H 10400 5600 50  0001 C CNN
 	1    10400 5600
@@
 F 0 "R8" V 3480 6850 50  0000 C CNN
 F 1 "1k" V 3400 6850 50  0000 C CNN
-F 2 "Resistor_SMD:R_0805_2012Metric" V 3330 6850 50  0001 C CNN
+F 2 "LeoDJ-kicad:R_0805_2012Metric" V 3330 6850 50  0001 C CNN
 F 3 "" H 3400 6850 50  0001 C CNN
 	1    3400 6850
@@
 F 0 "C3" H 3125 5800 50  0000 L CNN
 F 1 "100n" H 3125 5600 50  0000 L CNN
-F 2 "Capacitor_SMD:C_0805_2012Metric" H 3138 5550 50  0001 C CNN
+F 2 "LeoDJ-kicad:C_0805_2012Metric" H 3138 5550 50  0001 C CNN
 F 3 "" H 3100 5700 50  0001 C CNN
 	1    3100 5700
@@
 F 0 "R7" V 3480 5700 50  0000 C CNN
 F 1 "100" V 3400 5700 50  0000 C CNN
-F 2 "Resistor_SMD:R_0805_2012Metric" V 3330 5700 50  0001 C CNN
+F 2 "LeoDJ-kicad:R_0805_2012Metric" V 3330 5700 50  0001 C CNN
 F 3 "" H 3400 5700 50  0001 C CNN
 	1    3400 5700
@@
 F 0 "R6" V 680 7400 50  0000 C CNN
 F 1 "2k2" V 600 7400 50  0000 C CNN
-F 2 "Resistor_SMD:R_0805_2012Metric" V 530 7400 50  0001 C CNN
+F 2 "LeoDJ-kicad:R_0805_2012Metric" V 530 7400 50  0001 C CNN
 F 3 "" H 600 7400 50  0001 C CNN
 	1    600  7400
@@
 F 0 "C4" H 2225 6350 50  0000 L CNN
 F 1 "10µF" H 2225 6150 50  0000 L CNN
-F 2 "Capacitor_SMD:C_0805_2012Metric" H 2238 6100 50  0001 C CNN
+F 2 "LeoDJ-kicad:C_0805_2012Metric" H 2238 6100 50  0001 C CNN
 F 3 "" H 2200 6250 50  0001 C CNN
 	1    2200 6250
@@
 F 0 "C5" H 1525 6900 50  0000 L CNN
 F 1 "100n" H 1525 6700 50  0000 L CNN
-F 2 "Capacitor_SMD:C_0805_2012Metric" H 1538 6650 50  0001 C CNN
+F 2 "LeoDJ-kicad:C_0805_2012Metric" H 1538 6650 50  0001 C CNN
 F 3 "" H 1500 6800 50  0001 C CNN
 	1    1500 6800
@@
 F 0 "C6" H 4625 6450 50  0000 L CNN
 F 1 "100nF" H 4625 6250 50  0000 L CNN
-F 2 "Capacitor_SMD:C_0805_2012Metric" H 4638 6200 50  0001 C CNN
+F 2 "LeoDJ-kicad:C_0805_2012Metric" H 4638 6200 50  0001 C CNN
 F 3 "" H 4600 6350 50  0001 C CNN
 	1    4600 6350
@@
 F 0 "R9" V 5880 6900 50  0000 C CNN
 F 1 "56k" V 5800 6900 50  0000 C CNN
-F 2 "Resistor_SMD:R_0805_2012Metric" V 5730 6900 50  0001 C CNN
+F 2 "LeoDJ-kicad:R_0805_2012Metric" V 5730 6900 50  0001 C CNN
 F 3 "" H 5800 6900 50  0001 C CNN
 	1    5800 6900
@@
 F 0 "R10" V 5880 7300 50  0000 C CNN
 F 1 "10k" V 5800 7300 50  0000 C CNN
-F 2 "Resistor_SMD:R_0805_2012Metric" V 5730 7300 50  0001 C CNN
+F 2 "LeoDJ-kicad:R_0805_2012Metric" V 5730 7300 50  0001 C CNN
 F 3 "" H 5800 7300 50  0001 C CNN
 	1    5800 7300
@@
 F 0 "R11" V 980 2500 50  0000 C CNN
 F 1 "10k" V 900 2500 50  0000 C CNN
-F 2 "Resistor_SMD:R_0805_2012Metric" V 830 2500 50  0001 C CNN
+F 2 "LeoDJ-kicad:R_0805_2012Metric" V 830 2500 50  0001 C CNN
 F 3 "" H 900 2500 50  0001 C CNN
 	1    900  2500
@@
 F 0 "C10" H 9675 950 50  0000 L CNN
 F 1 "10µF" H 9675 750 50  0000 L CNN
-F 2 "Capacitor_SMD:C_0805_2012Metric" H 9688 700 50  0001 C CNN
+F 2 "LeoDJ-kicad:C_0805_2012Metric" H 9688 700 50  0001 C CNN
 F 3 "" H 9650 850 50  0001 C CNN
 	1    9650 850
@@
 F 0 "R12" H 4070 1096 50  0000 L CNN
 F 1 "10k" H 4070 1005 50  0000 L CNN
-F 2 "Resistor_SMD:R_0805_2012Metric" V 3930 1050 50  0001 C CNN
+F 2 "LeoDJ-kicad:R_0805_2012Metric" V 3930 1050 50  0001 C CNN
 F 3 "~" H 4000 1050 50  0001 C CNN
 	1    4000 1050
@@
 F 0 "R13" H 4320 1096 50  0000 L CNN
 F 1 "10k" H 4320 1005 50  0000 L CNN
-F 2 "Resistor_SMD:R_0805_2012Metric" V 4180 1050 50  0001 C CNN
+F 2 "LeoDJ-kicad:R_0805_2012Metric" V 4180 1050 50  0001 C CNN
 F 3 "~" H 4250 1050 50  0001 C CNN
 	1    4250 1050
@@
 F 0 "R14" V 1893 6800 50  0000 C CNN
 F 1 "1k" V 1984 6800 50  0000 C CNN
-F 2 "Resistor_SMD:R_0805_2012Metric" V 2030 6800 50  0001 C CNN
+F 2 "LeoDJ-kicad:R_0805_2012Metric" V 2030 6800 50  0001 C CNN
 F 3 "~" H 2100 6800 50  0001 C CNN
 	1    2100 6800
@@
 F 0 "R15" H 8920 3646 50  0000 L CNN
 F 1 "120" H 8920 3555 50  0000 L CNN
-F 2 "Resistor_SMD:R_0805_2012Metric" V 8780 3600 50  0001 C CNN
+F 2 "LeoDJ-kicad:R_0805_2012Metric" V 8780 3600 50  0001 C CNN
 F 3 "~" H 8850 3600 50  0001 C CNN
 	1    8850 3600
@@
 F 0 "R21" H 4220 3296 50  0000 L CNN
 F 1 "47k/220k" H 4220 3205 50  0000 L CNN
-F 2 "Resistor_SMD:R_0805_2012Metric" V 4080 3250 50  0001 C CNN
+F 2 "LeoDJ-kicad:R_0805_2012Metric" V 4080 3250 50  0001 C CNN
 F 3 "~" H 4150 3250 50  0001 C CNN
 	1    4150 3250
@@
 F 0 "R22" H 4220 3596 50  0000 L CNN
 F 1 "22k" H 4220 3505 50  0000 L CNN
-F 2 "Resistor_SMD:R_0805_2012Metric" V 4080 3550 50  0001 C CNN
+F 2 "LeoDJ-kicad:R_0805_2012Metric" V 4080 3550 50  0001 C CNN
 F 3 "~" H 4150 3550 50  0001 C CNN
 	1    4150 3550
@@
 F 0 "R23" H 4770 4096 50  0000 L CNN
 F 1 "1k" H 4770 4005 50  0000 L CNN
-F 2 "Resistor_SMD:R_0805_2012Metric" V 4630 4050 50  0001 C CNN
+F 2 "LeoDJ-kicad:R_0805_2012Metric" V 4630 4050 50  0001 C CNN
 F 3 "~" H 4700 4050 50  0001 C CNN
 	1    4700 4050
@@
 F 0 "C11" H 9425 950 50  0000 L CNN
 F 1 "100n" H 9425 750 50  0000 L CNN
-F 2 "Capacitor_SMD:C_0805_2012Metric" H 9438 700 50  0001 C CNN
+F 2 "LeoDJ-kicad:C_0805_2012Metric" H 9438 700 50  0001 C CNN
 F 3 "" H 9400 850 50  0001 C CNN
 	1    9400 850
@@
 F 0 "R24" V 980 1550 50  0000 C CNN
 F 1 "10k" V 900 1550 50  0000 C CNN
-F 2 "Resistor_SMD:R_0805_2012Metric" V 830 1550 50  0001 C CNN
+F 2 "LeoDJ-kicad:R_0805_2012Metric" V 830 1550 50  0001 C CNN
 F 3 "" H 900 1550 50  0001 C CNN
 	1    900  1550
@@
 Text Notes 6050 4450 0    39   ~ 0
 MOSFETs can be optionally fitted\nFor that the trace bridging gate and source has to be cut\nIn the layout this is implemented manually
+$Comp
+L Graphic:Logo_Open_Hardware_Small LOGO1
+U 1 1 5B3753B8
+P 8850 6300
+F 0 "LOGO1" H 8850 6575 50  0001 C CNN
+F 1 "Logo_Open_Hardware_Small" H 8850 6075 50  0001 C CNN
+F 2 "Symbol:OSHW-Logo2_7.3x6mm_SilkScreen" H 8850 6300 50  0001 C CNN
+F 3 "~" H 8850 6300 50  0001 C CNN
+	1    8850 6300
+	1    0    0    -1
+$EndComp
+$Comp
+L Graphic:SYM_Arrow_Tiny SYM1
+U 1 1 5B37639E
+P 9250 6300
+F 0 "SYM1" H 9250 6360 50  0001 C CNN
+F 1 "SYM_Arrow_Tiny" H 9260 6250 50  0001 C CNN
+F 2 "leodj-kicad:Otter_Lightbulb_smaller" H 9250 6300 50  0001 C CNN
+F 3 "~" H 9250 6300 50  0001 C CNN
+	1    9250 6300
+	1    0    0    -1
+$EndComp
+$Comp
+L Graphic:SYM_Arrow_Tiny SYM2
+U 1 1 5B3BA95F
+P 9250 6250
+F 0 "SYM2" H 9250 6310 50  0001 C CNN
+F 1 "SYM_Arrow_Tiny" H 9260 6200 50  0001 C CNN
+F 2 "leodj-kicad:QR_Code_SHMod24" H 9250 6250 50  0001 C CNN
+F 3 "~" H 9250 6250 50  0001 C CNN
+	1    9250 6250
+	1    0    0    -1
+$EndComp
+Text Notes 9250 6400 0    50   ~ 0
+^ Logos
 $EndSCHEMATC

Commit message: add RS485 connector markings
Parts:
- added J8: GND, TestPoint:TestPoint_Pad_D1.0mm, symbol SHMod24-rescue:Conn_01x01-Connector_Generic
Changed lines of the file:
@@
 Text Notes 9250 6400 0    50   ~ 0
 ^ Logos
+$Comp
+L SHMod24-rescue:Conn_01x01-Connector_Generic J8
+U 1 1 5B3D026A
+P 2200 900
+F 0 "J8" H 2300 900 50  0000 C CNN
+F 1 "GND" H 2150 1000 50  0000 C CNN
+F 2 "TestPoint:TestPoint_Pad_D1.0mm" H 2200 900 50  0001 C CNN
+F 3 "~" H 2200 900 50  0001 C CNN
+	1    2200 900
+	-1   0    0    1
+$EndComp
+$Comp
+L power:GND #PWR0133
+U 1 1 5B3D04C5
+P 2400 900
+F 0 "#PWR0133" H 2400 650 50  0001 C CNN
+F 1 "GND" H 2405 727 50  0000 C CNN
+F 2 "" H 2400 900 50  0001 C CNN
+F 3 "" H 2400 900 50  0001 C CNN
+	1    2400 900
+	1    0    0    -1
+$EndComp
 $EndSCHEMATC
